File: Ram16/Ram16.kicad_sch (KiCad schematic)
At the start: 18 parts, among them J1 Conn_01x03, J10 Conn_01x16, J11 Conn_01x16, J2 Conn_01x08, J3 Conn_01x08, J4 Conn_01x08, J5 Conn_01x08, J6 Conn_01x02, J7 Conn_01x02, J8 Conn_01x02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

Commit message: Added cappacitor to all Schematic
Parts:
- added C1, C2: 0.1uf, symbol Device:C
Connections:
- net at J1.3 (Pin_3), J8.1 (Pin_1), J9.1 (Pin_1)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: now also C1.1, C2.1
- net at J1.1 (Pin_1), J8.2 (Pin_2), J9.2 (Pin_2)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: now also C1.2, C2.2
Changed lines of the file:
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@@
   (junction (at 91.44 40.64) (diameter 0) (color 0 0 0 0)
   )
+  (junction (at 106.68 137.16) (diameter 0) (color 0 0 0 0)
+  )
   (junction (at 195.58 85.09) (diameter 0) (color 0 0 0 0)
   )
@@
   (junction (at 68.58 53.34) (diameter 0) (color 0 0 0 0)
   )
+  (junction (at 106.68 129.54) (diameter 0) (color 0 0 0 0)
+  )
   (junction (at 247.65 143.51) (diameter 0) (color 0 0 0 0)
   )
@@
   )
   (junction (at 81.28 40.64) (diameter 0) (color 0 0 0 0)
+  )
+  (junction (at 115.57 137.16) (diameter 0) (color 0 0 0 0)
   )
   (junction (at 134.62 147.32) (diameter 0) (color 0 0 0 0)
@@
     (stroke (width 0) (type default))
   )
+  (wire (pts (xy 106.68 137.16) (xy 115.57 137.16))
+    (stroke (width 0) (type default))
+  )
   (wire (pts (xy 154.94 97.79) (xy 154.94 48.26))
     (stroke (width 0) (type default))
@@
     (stroke (width 0) (type default))
   )
+  (wire (pts (xy 115.57 137.16) (xy 137.16 137.16))
+    (stroke (width 0) (type default))
+  )
   (wire (pts (xy 57.15 173.99) (xy 34.29 173.99))
     (stroke (width 0) (type default))
@@
     (stroke (width 0) (type default))
   )
+  (wire (pts (xy 101.6 129.54) (xy 106.68 129.54))
+    (stroke (width 0) (type default))
+  )
   (wire (pts (xy 195.58 118.11) (xy 234.95 118.11))
     (stroke (width 0) (type default))
@@
     (stroke (width 0) (type default))
   )
-  (wire (pts (xy 99.06 137.16) (xy 137.16 137.16))
+  (wire (pts (xy 99.06 137.16) (xy 106.68 137.16))
     (stroke (width 0) (type default))
   )
@@
   )
   (wire (pts (xy 139.7 73.66) (xy 234.95 73.66))
+    (stroke (width 0) (type default))
+  )
+  (wire (pts (xy 106.68 129.54) (xy 115.57 129.54))
     (stroke (width 0) (type default))
   )
@@
     )
   )
+  (symbol (lib_id "Device:C") (at 115.57 133.35 0) (unit 1)
+    (in_bom yes) (on_board yes) (dnp no)
+    (property "Reference" "C2" (at 116.84 130.81 0)
+      (effects (font (size 1.27 1.27)) (justify left))
+    )
+    (property "Value" "0.1uf" (at 116.84 135.89 0)
+      (effects (font (size 1.27 1.27)) (justify left))
+    )
+    (property "Footprint" "" (at 116.5352 137.16 0)
+      (effects (font (size 1.27 1.27)) hide)
+    )
+    (property "Datasheet" "~" (at 115.57 133.35 0)
+      (effects (font (size 1.27 1.27)) hide)
+    )
+    (pin "1")
+    (pin "2")
+    (instances
+      (project "Ram16"
+        (path "/d849d05f-2032-4b50-8296-fc02fbafeedb"
+          (reference "C2") (unit 1)
+        )
+      )
+    )
+  )
   (symbol (lib_id "Connector_Generic:Conn_01x02") (at 21.59 158.75 180) (unit 1)
     (in_bom yes) (on_board yes) (dnp no) (fields_autoplaced)
@@
         )
       )
+    )
+  )
+  (symbol (lib_id "Device:C") (at 106.68 133.35 0) (unit 1)
+    (in_bom yes) (on_board yes) (dnp no)
+    (property "Reference" "C1" (at 107.95 130.81 0)
+      (effects (font (size 1.27 1.27)) (justify left))
+    )
+    (property "Value" "0.1uf" (at 107.95 135.89 0)
+      (effects (font (size 1.27 1.27)) (justify left))
+    )
+    (property "Footprint" "" (at 107.6452 137.16 0)
+      (effects (font (size 1.27 1.27)) hide)
+    )
+    (property "Datasheet" "~" (at 106.68 133.35 0)
+      (effects (font (size 1.27 1.27)) hide)
+    )
+    (pin "1")
+    (pin "2")
+    (instances
+      (project "Ram16"
+        (path "/d849d05f-2032-4b50-8296-fc02fbafeedb"
+          (reference "C1") (unit 1)
+        )
+      )

Commit message: Started assigning footprint
Parts:
- C1, C2: footprint (none) -> Capacitor_SMD:C_0603_1608Metric_Pad1.08x0.95mm_HandSolder
- J1: footprint (none) -> Connector_PinHeader_2.54mm:PinHeader_1x03_P2.54mm_Vertical
- J10, J11: footprint (none) -> Connector_PinHeader_2.54mm:PinHeader_1x16_P2.54mm_Vertical
- J2, J3, J4, J5: footprint (none) -> Connector_PinHeader_2.54mm:PinHeader_1x08_P2.54mm_Vertical
- J6, J7, J8, J9: footprint (none) -> Connector_PinHeader_2.54mm:PinHeader_1x02_P2.54mm_Vertical
- U2, U3: footprint (none) -> Package_TO_SOT_SMD:SOT-353_SC-70-5_Handsoldering
- U23, U24: footprint (none) -> Package_SO:SSOP-28_5.3x10.2mm_P0.65mm
- U5, U6: footprint (none) -> Package_SO:SOIC-14W_7.5x9mm_P1.27mm
- U7: footprint (none) -> Package_SO:TSOP-5_1.65x3.05mm_P0.95mm
Changed lines of the file:
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@@
       (effects (font (size 1.27 1.27)) hide)
     )
-    (property "Footprint" "" (at 78.74 129.54 0)
+    (property "Footprint" "Connector_PinHeader_2.54mm:PinHeader_1x02_P2.54mm_Vertical" (at 78.74 129.54 0)
       (effects (font (size 1.27 1.27)) hide)
     )
@@
       (effects (font (size 1.27 1.27)))
     )
-    (property "Footprint" "" (at 116.84 83.82 0)
+    (property "Footprint" "Package_SO:SSOP-28_5.3x10.2mm_P0.65mm" (at 116.84 83.82 0)
       (effects (font (size 1.27 1.27)) hide)
     )
@@
       (effects (font (size 1.27 1.27)) (justify left) hide)
     )
-    (property "Footprint" "" (at 276.86 118.11 0)
+    (property "Footprint" "Connector_PinHeader_2.54mm:PinHeader_1x08_P2.54mm_Vertical" (at 276.86 118.11 0)
       (effects (font (size 1.27 1.27)) hide)
     )
@@
       (effects (font (size 1.27 1.27)) (justify left))
     )
-    (property "Footprint" "" (at 247.65 71.12 0)
+    (property "Footprint" "Package_SO:SOIC-14W_7.5x9mm_P1.27mm" (at 247.65 71.12 0)
       (effects (font (size 1.27 1.27)) hide)
     )
@@
       (effects (font (size 1.27 1.27)) (justify left))
     )
-    (property "Footprint" "" (at 116.5352 137.16 0)
+    (property "Footprint" "Capacitor_SMD:C_0603_1608Metric_Pad1.08x0.95mm_HandSolder" (at 116.5352 137.16 0)
       (effects (font (size 1.27 1.27)) hide)
     )
@@
       (effects (font (size 1.27 1.27)) hide)
     )
-    (property "Footprint" "" (at 21.59 158.75 0)
+    (property "Footprint" "Connector_PinHeader_2.54mm:PinHeader_1x02_P2.54mm_Vertical" (at 21.59 158.75 0)
       (effects (font (size 1.27 1.27)) hide)
     )
@@
       (effects (font (size 1.27 1.27)) hide)
     )
-    (property "Footprint" "" (at 29.21 158.75 0)
+    (property "Footprint" "Connector_PinHeader_2.54mm:PinHeader_1x02_P2.54mm_Vertical" (at 29.21 158.75 0)
       (effects (font (size 1.27 1.27)) hide)
     )
@@
       (effects (font (size 1.27 1.27)) hide)
     )
-    (property "Footprint" "" (at 90.17 129.54 0)
+    (property "Footprint" "Connector_PinHeader_2.54mm:PinHeader_1x02_P2.54mm_Vertical" (at 90.17 129.54 0)
       (effects (font (size 1.27 1.27)) hide)
     )
@@
       (effects (font (size 1.27 1.27)) (justify left))
     )
-    (property "Footprint" "" (at 247.65 123.19 0)
+    (property "Footprint" "Package_SO:SOIC-14W_7.5x9mm_P1.27mm" (at 247.65 123.19 0)
       (effects (font (size 1.27 1.27)) hide)
     )
@@
       (effects (font (size 1.27 1.27)) (justify left) hide)
     )
-    (property "Footprint" "" (at 265.43 66.04 0)
+    (property "Footprint" "Connector_PinHeader_2.54mm:PinHeader_1x08_P2.54mm_Vertical" (at 265.43 66.04 0)
       (effects (font (size 1.27 1.27)) hide)
     )
@@
       (effects (font (size 1.27 1.27)))
     )
-    (property "Footprint" "" (at 72.39 173.99 0)
+    (property "Footprint" "Package_TO_SOT_SMD:SOT-353_SC-70-5_Handsoldering" (at 72.39 173.99 0)
       (effects (font (size 1.27 1.27)) hide)
     )
@@
       (effects (font (size 1.27 1.27)))
     )
-    (property "Footprint" "" (at 72.39 147.32 0)
+    (property "Footprint" "Package_TO_SOT_SMD:SOT-353_SC-70-5_Handsoldering" (at 72.39 147.32 0)
       (effects (font (size 1.27 1.27)) hide)
     )
@@
       (effects (font (size 1.27 1.27)) (justify left))
     )
-    (property "Footprint" "" (at 107.6452 137.16 0)
+    (property "Footprint" "Capacitor_SMD:C_0603_1608Metric_Pad1.08x0.95mm_HandSolder" (at 107.6452 137.16 0)
       (effects (font (size 1.27 1.27)) hide)
     )
@@
       (effects (font (size 1.27 1.27)) (justify left) hide)
     )
-    (property "Footprint" "" (at 265.43 118.11 0)
+    (property "Footprint" "Connector_PinHeader_2.54mm:PinHeader_1x08_P2.54mm_Vertical" (at 265.43 118.11 0)
       (effects (font (size 1.27 1.27)) hide)
     )
@@
       (effects (font (size 1.27 1.27)) hide)
     )
-    (property "Footprint" "" (at 86.36 26.67 0)
+    (property "Footprint" "Connector_PinHeader_2.54mm:PinHeader_1x16_P2.54mm_Vertical" (at 86.36 26.67 0)
       (effects (font (size 1.27 1.27)) hide)
     )
@@
       (effects (font (size 1.27 1.27)) hide)
     )
-    (property "Footprint" "" (at 125.73 125.73 0)
+    (property "Footprint" "Connector_PinHeader_2.54mm:PinHeader_1x03_P2.54mm_Vertical" (at 125.73 125.73 0)
       (effects (font (size 1.27 1.27)) hide)
     )
@@
       (effects (font (size 1.27 1.27)) hide)
     )
-    (property "Footprint" "" (at 86.36 35.56 0)
+    (property "Footprint" "Connector_PinHeader_2.54mm:PinHeader_1x16_P2.54mm_Vertical" (at 86.36 35.56 0)
       (effects (font (size 1.27 1.27)) hide)
     )
@@
       (effects (font (size 1.27 1.27)) (justify left) hide)
     )
-    (property "Footprint" "" (at 276.86 66.04 0)
+    (property "Footprint" "Connector_PinHeader_2.54mm:PinHeader_1x08_P2.54mm_Vertical" (at 276.86 66.04 0)
       (effects (font (size 1.27 1.27)) hide)
     )
@@
       (effects (font (size 1.27 1.27)))
     )
-    (property "Footprint" "" (at 180.34 83.82 0)
+    (property "Footprint" "Package_SO:SSOP-28_5.3x10.2mm_P0.65mm" (at 180.34 83.82 0)
       (effects (font (size 1.27 1.27)) hide)
     )
@@
       (effects (font (size 1.27 1.27)))
     )
-    (property "Footprint" "" (at 207.01 154.94 0)
-      (effects (font (size 1.27 1.27)) hide)
-    )
+    (property "Footprint" "Package_SO:TSOP-5_1.65x3.05mm_P0.95mm" (at 207.01 154.94 0)
+      (effects (font (size 1.27 1.27)) hide)
+    )
