File: ALU/ALU.kicad_sch (KiCad schematic)
At the start: 29 parts, among them J26 Conn_01x08, J27 Conn_01x08, J28 Conn_01x08, J29 Conn_01x08, J32 Conn_01x08, J33 Conn_01x08, J5 Conn_01x05, J51 Conn_01x02, J52 Conn_01x02, J6 Conn_01x05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

Commit message: Updated Footprint
Parts:
- C7, C8: footprint (none) -> Capacitor_SMD:C_0603_1608Metric_Pad1.08x0.95mm_HandSolder
- D22, D23, D24, D25, D26, D27, D28, D29: footprint (none) -> LED_THT:LED_D5.0mm-3
- J26, J27, J28, J29, J32, J33: footprint (none) -> Connector_PinHeader_2.54mm:PinHeader_1x08_P2.54mm_Vertical
- J5, J6: footprint (none) -> Connector_PinHeader_2.54mm:PinHeader_1x05_P2.54mm_Vertical
- J51, J52: footprint (none) -> Connector_PinHeader_2.54mm:PinHeader_1x02_P2.54mm_Vertical
- U17, U18: footprint (none) -> Package_SO:SOIC-16_3.9x9.9mm_P1.27mm
- U19, U20, U8: footprint (none) -> Package_SO:SOIC-14_3.9x8.7mm_P1.27mm
- U5: footprint (none) -> Package_SO:TSOP-5_1.65x3.05mm_P0.95mm
- U6: footprint (none) -> Package_SO:TSSOP-14_4.4x5mm_P0.65mm
- U7: footprint (none) -> Package_SO:SOIC-14W_7.5x9mm_P1.27mm
