File: BusInput/BusInput.kicad_sch (KiCad schematic)
At the start: 4 parts, among them J1 Conn_01x02, J2 Conn_01x08, J3 Conn_01x02, SW1 SW_DIP_x08

Commit message: Updated Footprint
Parts:
- J1, J3: footprint (none) -> Connector_PinHeader_2.54mm:PinHeader_1x02_P2.54mm_Vertical
- J2: footprint (none) -> Connector_PinHeader_2.54mm:PinHeader_1x08_P2.54mm_Vertical
- SW1: footprint (none) -> Package_DIP:DIP-8_W8.89mm_SMDSocket_LongPads
Changed lines of the file:
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@@
       (effects (font (size 1.27 1.27)) (justify left) hide)
     )
-    (property "Footprint" "" (at 137.16 67.31 0)
+    (property "Footprint" "Package_DIP:DIP-8_W8.89mm_SMDSocket_LongPads" (at 137.16 67.31 0)
       (effects (font (size 1.27 1.27)) hide)
     )
@@
       (effects (font (size 1.27 1.27)) (justify left) hide)
     )
-    (property "Footprint" "" (at 161.29 91.44 0)
+    (property "Footprint" "Connector_PinHeader_2.54mm:PinHeader_1x02_P2.54mm_Vertical" (at 161.29 91.44 0)
       (effects (font (size 1.27 1.27)) hide)
     )
@@
       (effects (font (size 1.27 1.27)) hide)
     )
-    (property "Footprint" "" (at 139.7 80.01 0)
+    (property "Footprint" "Connector_PinHeader_2.54mm:PinHeader_1x08_P2.54mm_Vertical" (at 139.7 80.01 0)
       (effects (font (size 1.27 1.27)) hide)
     )
@@
       (effects (font (size 1.27 1.27)) (justify left) hide)
     )
-    (property "Footprint" "" (at 161.29 80.01 0)
+    (property "Footprint" "Connector_PinHeader_2.54mm:PinHeader_1x02_P2.54mm_Vertical" (at 161.29 80.01 0)
       (effects (font (size 1.27 1.27)) hide)
     )
