File: Register8/Register8.kicad_sch (KiCad schematic)
At the start: 21 parts, among them J1 Conn_01x08, J2 Conn_01x08, J3 Conn_01x08, J4 Conn_01x08, J5 Conn_01x04, J6 Conn_01x04, J7 Conn_01x02, J8 Conn_01x02, U1 74HC245, U2 74LS173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

Commit message: Added cappacitor to all Schematic
Parts:
- added C1, C2: 0.1uf, symbol Device:C
Connections:
- net at J7.1 (Pin_1), J8.1 (Pin_1), RN1.1 (common)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: now also C1.2, C2.2
- net at J7.2 (Pin_2), J8.2 (Pin_2), U1.1 (A->B)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: now also C1.1, C2.1
Changed lines of the file:
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@@
   (junction (at 92.71 148.59) (diameter 0) (color 0 0 0 0)
   )
+  (junction (at 55.88 82.55) (diameter 0) (color 0 0 0 0)
+  )
   (junction (at 48.26 39.37) (diameter 0) (color 0 0 0 0)
   )
@@
   (junction (at 162.56 82.55) (diameter 0) (color 0 0 0 0)
   )
+  (junction (at 48.26 90.17) (diameter 0) (color 0 0 0 0)
+  )
   (junction (at 87.63 146.05) (diameter 0) (color 0 0 0 0)
   )
@@
   (junction (at 60.96 31.75) (diameter 0) (color 0 0 0 0)
   )
+  (junction (at 55.88 90.17) (diameter 0) (color 0 0 0 0)
+  )
+  (junction (at 66.04 82.55) (diameter 0) (color 0 0 0 0)
+  )
   (junction (at 102.87 154.94) (diameter 0) (color 0 0 0 0)
   )
@@
     (stroke (width 0) (type default))
   )
+  (wire (pts (xy 55.88 82.55) (xy 66.04 82.55))
+    (stroke (width 0) (type default))
+  )
   (wire (pts (xy 162.56 82.55) (xy 162.56 62.23))
     (stroke (width 0) (type default))
@@
     (stroke (width 0) (type default))
   )
+  (wire (pts (xy 48.26 90.17) (xy 48.26 85.09))
+    (stroke (width 0) (type default))
+  )
   (wire (pts (xy 241.3 31.75) (xy 102.87 31.75))
     (stroke (width 0) (type default))
@@
     (stroke (width 0) (type default))
   )
+  (wire (pts (xy 55.88 90.17) (xy 66.04 90.17))
+    (stroke (width 0) (type default))
+  )
   (wire (pts (xy 238.76 34.29) (xy 100.33 34.29))
     (stroke (width 0) (type default))
@@
     (stroke (width 0) (type default))
   )
+  (wire (pts (xy 66.04 82.55) (xy 77.47 82.55))
+    (stroke (width 0) (type default))
+  )
   (wire (pts (xy 87.63 104.14) (xy 87.63 146.05))
     (stroke (width 0) (type default))
@@
     (stroke (width 0) (type default))
   )
-  (wire (pts (xy 48.26 82.55) (xy 77.47 82.55))
+  (wire (pts (xy 48.26 82.55) (xy 55.88 82.55))
     (stroke (width 0) (type default))
   )
@@
     (stroke (width 0) (type default))
   )
-  (wire (pts (xy 48.26 114.3) (xy 48.26 85.09))
+  (wire (pts (xy 48.26 114.3) (xy 48.26 90.17))
     (stroke (width 0) (type default))
   )
@@
   )
   (wire (pts (xy 162.56 82.55) (xy 165.1 82.55))
+    (stroke (width 0) (type default))
+  )
+  (wire (pts (xy 48.26 90.17) (xy 55.88 90.17))
     (stroke (width 0) (type default))
   )
@@
     )
   )
+  (symbol (lib_id "Device:C") (at 66.04 86.36 0) (unit 1)
+    (in_bom yes) (on_board yes) (dnp no)
+    (property "Reference" "C2" (at 66.04 83.82 0)
+      (effects (font (size 1.27 1.27)) (justify left))
+    )
+    (property "Value" "0.1uf" (at 67.31 88.9 0)
+      (effects (font (size 1.27 1.27)) (justify left))
+    )
+    (property "Footprint" "" (at 67.0052 90.17 0)
+      (effects (font (size 1.27 1.27)) hide)
+    )
+    (property "Datasheet" "~" (at 66.04 86.36 0)
+      (effects (font (size 1.27 1.27)) hide)
+    )
+    (pin "1")
+    (pin "2")
+    (instances
+      (project "Register8"
+        (path "/5cfd5bcb-044d-4fc2-a5e2-246a2c9e17c3"
+          (reference "C2") (unit 1)
+        )
+      )
+    )
+  )
   (symbol (lib_id "Device:LED") (at 97.79 154.94 90) (unit 1)
     (in_bom yes) (on_board yes) (dnp no)
@@
         )
       )
+    )
+  )
+  (symbol (lib_id "Device:C") (at 55.88 86.36 0) (unit 1)
+    (in_bom yes) (on_board yes) (dnp no)
+    (property "Reference" "C1" (at 55.88 83.82 0)
+      (effects (font (size 1.27 1.27)) (justify left))
+    )
+    (property "Value" "0.1uf" (at 57.15 88.9 0)
+      (effects (font (size 1.27 1.27)) (justify left))
+    )
+    (property "Footprint" "" (at 56.8452 90.17 0)
+      (effects (font (size 1.27 1.27)) hide)
+    )
+    (property "Datasheet" "~" (at 55.88 86.36 0)
+      (effects (font (size 1.27 1.27)) hide)
+    )
+    (pin "1")
+    (pin "2")
+    (instances
+      (project "Register8"
+        (path "/5cfd5bcb-044d-4fc2-a5e2-246a2c9e17c3"
+          (reference "C1") (unit 1)
+        )
+      )

Commit message: Started assigning footprint
Parts:
- C1, C2: footprint (none) -> Capacitor_SMD:C_0603_1608Metric_Pad1.08x0.95mm_HandSolder
- D1, D2, D3, D4, D5, D6, D7, D8: footprint (none) -> LED_THT:LED_D5.0mm-3
- J1, J2, J3, J4: footprint (none) -> Connector_PinHeader_2.54mm:PinHeader_1x08_P2.54mm_Vertical
- J5, J6: footprint (none) -> Connector_PinHeader_2.54mm:PinHeader_1x04_P2.54mm_Vertical
- J7, J8: footprint (none) -> Connector_PinHeader_2.54mm:PinHeader_1x02_P2.54mm_Vertical
- U1: footprint (none) -> Package_SO:SOIC-14W_7.5x9mm_P1.27mm
- U2, U3: footprint (none) -> Package_SO:SOIC-16_3.9x9.9mm_P1.27mm
- U4: footprint (none) -> Package_SO:TSOP-5_1.65x3.05mm_P0.95mm
Changed lines of the file:
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@@
       (effects (font (size 1.27 1.27)) (justify left))
     )
-    (property "Footprint" "" (at 170.18 95.25 0)
+    (property "Footprint" "Package_SO:SOIC-16_3.9x9.9mm_P1.27mm" (at 170.18 95.25 0)
       (effects (font (size 1.27 1.27)) hide)
     )
@@
       (effects (font (size 1.27 1.27)) (justify right) hide)
     )
-    (property "Footprint" "" (at 85.09 148.59 0)
+    (property "Footprint" "LED_THT:LED_D5.0mm-3" (at 85.09 148.59 0)
       (effects (font (size 1.27 1.27)) hide)
     )
@@
       (effects (font (size 1.27 1.27)) (justify left))
     )
-    (property "Footprint" "" (at 226.06 95.25 0)
+    (property "Footprint" "Package_SO:SOIC-16_3.9x9.9mm_P1.27mm" (at 226.06 95.25 0)
       (effects (font (size 1.27 1.27)) hide)
     )
@@
       (effects (font (size 1.27 1.27)))
     )
-    (property "Footprint" "" (at 97.79 91.44 0)
+    (property "Footprint" "Package_SO:SOIC-14W_7.5x9mm_P1.27mm" (at 97.79 91.44 0)
       (effects (font (size 1.27 1.27)) hide)
     )
@@
       (effects (font (size 1.27 1.27)) hide)
     )
-    (property "Footprint" "" (at 30.48 85.09 0)
+    (property "Footprint" "Connector_PinHeader_2.54mm:PinHeader_1x02_P2.54mm_Vertical" (at 30.48 85.09 0)
       (effects (font (size 1.27 1.27)) hide)
     )
@@
       (effects (font (size 1.27 1.27)) (justify left))
     )
-    (property "Footprint" "" (at 67.0052 90.17 0)
+    (property "Footprint" "Capacitor_SMD:C_0603_1608Metric_Pad1.08x0.95mm_HandSolder" (at 67.0052 90.17 0)
       (effects (font (size 1.27 1.27)) hide)
     )
@@
       (effects (font (size 1.27 1.27)) (justify right) hide)
     )
-    (property "Footprint" "" (at 97.79 154.94 0)
+    (property "Footprint" "LED_THT:LED_D5.0mm-3" (at 97.79 154.94 0)
       (effects (font (size 1.27 1.27)) hide)
     )
@@
       (effects (font (size 1.27 1.27)) (justify right) hide)
     )
-    (property "Footprint" "" (at 87.63 149.86 0)
+    (property "Footprint" "LED_THT:LED_D5.0mm-3" (at 87.63 149.86 0)
       (effects (font (size 1.27 1.27)) hide)
     )
@@
       (effects (font (size 1.27 1.27)) hide)
     )
-    (property "Footprint" "" (at 43.18 64.77 0)
+    (property "Footprint" "Connector_PinHeader_2.54mm:PinHeader_1x04_P2.54mm_Vertical" (at 43.18 64.77 0)
       (effects (font (size 1.27 1.27)) hide)
     )
@@
       (effects (font (size 1.27 1.27)))
     )
-    (property "Footprint" "" (at 135.89 62.23 0)
+    (property "Footprint" "Package_SO:TSOP-5_1.65x3.05mm_P0.95mm" (at 135.89 62.23 0)
       (effects (font (size 1.27 1.27)) hide)
     )
@@
       (effects (font (size 1.27 1.27)) hide)
     )
-    (property "Footprint" "" (at 55.88 41.91 0)
+    (property "Footprint" "Connector_PinHeader_2.54mm:PinHeader_1x08_P2.54mm_Vertical" (at 55.88 41.91 0)
       (effects (font (size 1.27 1.27)) hide)
     )
@@
       (effects (font (size 1.27 1.27)) hide)
     )
-    (property "Footprint" "" (at 30.48 64.77 0)
+    (property "Footprint" "Connector_PinHeader_2.54mm:PinHeader_1x04_P2.54mm_Vertical" (at 30.48 64.77 0)
       (effects (font (size 1.27 1.27)) hide)
     )
@@
       (effects (font (size 1.27 1.27)) hide)
     )
-    (property "Footprint" "" (at 43.18 41.91 0)
+    (property "Footprint" "Connector_PinHeader_2.54mm:PinHeader_1x08_P2.54mm_Vertical" (at 43.18 41.91 0)
       (effects (font (size 1.27 1.27)) hide)
     )
@@
       (effects (font (size 1.27 1.27)) (justify right) hide)
     )
-    (property "Footprint" "" (at 92.71 152.4 0)
+    (property "Footprint" "LED_THT:LED_D5.0mm-3" (at 92.71 152.4 0)
       (effects (font (size 1.27 1.27)) hide)
     )
@@
       (effects (font (size 1.27 1.27)) (justify right) hide)
     )
-    (property "Footprint" "" (at 90.17 151.13 0)
+    (property "Footprint" "LED_THT:LED_D5.0mm-3" (at 90.17 151.13 0)
       (effects (font (size 1.27 1.27)) hide)
     )
@@
       (effects (font (size 1.27 1.27)) (justify right) hide)
     )
-    (property "Footprint" "" (at 102.87 158.75 0)
+    (property "Footprint" "LED_THT:LED_D5.0mm-3" (at 102.87 158.75 0)
       (effects (font (size 1.27 1.27)) hide)
     )
@@
       (effects (font (size 1.27 1.27)) hide)
     )
-    (property "Footprint" "" (at 68.58 41.91 0)
+    (property "Footprint" "Connector_PinHeader_2.54mm:PinHeader_1x08_P2.54mm_Vertical" (at 68.58 41.91 0)
       (effects (font (size 1.27 1.27)) hide)
     )
@@
       (effects (font (size 1.27 1.27)) (justify right) hide)
     )
-    (property "Footprint" "" (at 95.25 153.67 0)
+    (property "Footprint" "LED_THT:LED_D5.0mm-3" (at 95.25 153.67 0)
       (effects (font (size 1.27 1.27)) hide)
     )
@@
       (effects (font (size 1.27 1.27)) (justify left))
     )
-    (property "Footprint" "" (at 56.8452 90.17 0)
+    (property "Footprint" "Capacitor_SMD:C_0603_1608Metric_Pad1.08x0.95mm_HandSolder" (at 56.8452 90.17 0)
       (effects (font (size 1.27 1.27)) hide)
     )
@@
       (effects (font (size 1.27 1.27)) (justify right) hide)
     )
-    (property "Footprint" "" (at 100.33 156.21 0)
+    (property "Footprint" "LED_THT:LED_D5.0mm-3" (at 100.33 156.21 0)
       (effects (font (size 1.27 1.27)) hide)
     )
@@
       (effects (font (size 1.27 1.27)) hide)
     )
-    (property "Footprint" "" (at 43.18 85.09 0)
+    (property "Footprint" "Connector_PinHeader_2.54mm:PinHeader_1x02_P2.54mm_Vertical" (at 43.18 85.09 0)
       (effects (font (size 1.27 1.27)) hide)
     )
@@
       (effects (font (size 1.27 1.27)) hide)
     )
-    (property "Footprint" "" (at 30.48 41.91 0)
-      (effects (font (size 1.27 1.27)) hide)
-    )
+    (property "Footprint" "Connector_PinHeader_2.54mm:PinHeader_1x08_P2.54mm_Vertical" (at 30.48 41.91 0)
+      (effects (font (size 1.27 1.27)) hide)
+    )

Commit message: Made 8Bit Register PCB
Parts:
- removed RN1: 220, Resistor_THT:R_Array_SIP9, symbol Device:R_Network08
- removed U4: 74AHC1G04, Package_SO:TSOP-5_1.65x3.05mm_P0.95mm, symbol 74xGxx:74AHC1G04
- added H1, H2, H3, H4: MountingHole, MountingHole:MountingHole_3.2mm_M3, symbol Mechanical:MountingHole
- added R1, R2, R3, R4, R5, R6, R7, R8: 220, Resistor_SMD:R_0805_2012Metric_Pad1.20x1.40mm_HandSolder, symbol Device:R
- C1, C2: footprint Capacitor_SMD:C_0603_1608Metric_Pad1.08x0.95mm_HandSolder -> Capacitor_SMD:C_0805_2012Metric_Pad1.18x1.45mm_HandSolder
- D1, D2, D3, D4, D5, D6, D7, D8: footprint LED_THT:LED_D5.0mm-3 -> LED_THT:LED_D5.0mm
- U1: footprint Package_SO:SOIC-14W_7.5x9mm_P1.27mm -> Package_SO:TSSOP-20_4.4x6.5mm_P0.65mm
Connections:
- net at C1.2, C2.2, J7.1 (Pin_1)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: now also R1.2, R2.2, R3.2, R4.2, R5.2, R6.2, R7.2, R8.2
- net at U2.10 (E2), U2.9 (E1), U3.10 (E2)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: now also J5.3 (Pin_3), J6.3 (Pin_3)
- net at D1.1 (K): now also R1.1
- net at D6.1 (K): now also R6.1
- net at D2.1 (K): now also R2.1
- net at D4.1 (K): now also R4.1
- net at D3.1 (K): now also R3.1
- net at D8.1 (K): now also R8.1
- net at D5.1 (K): now also R5.1
- net at D7.1 (K): now also R7.1
Other:
- note added: "8 0 Bit"
- note added: "Output Enable Input Enable / Clock Reset"
- note removed: "Output Enable Input Enable Clock Reset"
